File: Controller/Controller.kicad_pcb (KiCad board)
At the start: 2 copper layers, 114 x 50 mm, 57 parts, among them P11 CONN_SHOULDER, P3 MOUNT, P4 MOUNT, P5 MOUNT, P6 MOUNT, P7 MOUNT, P8 CONN_SHOULDER, Q1 DMN2050L, SW1 BUTTON, SW10 BUTTON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

Commit message: Improved traces in power supply circuit. Added clearance on inside of drill holes. Removed sharp inside corners and replaced with cirular cutouts. Removed removed pull-down resistors because I am using internal pull-ups and negative logic with buttons.
Parts:
- removed P11, P8: CONN_SHOULDER, Controller:CONN_SHOULDER_M
- removed R10, R11, R12, R13, R14, R15, R16, R17, R18, R19, R20, R6, R7, R8, R9: 10k, Resistors_SMD:R_0805
- added P1: CONN_SHOULDER, Controller:CONN_SHOULDER_M, F.Cu at (20.2, 16.9)
- added P2: CONN_SHOULDER, Controller:CONN_SHOULDER_M, F.Cu at (106.2, 16.9)
- moved P5 104.0 mm to (122.0, 54.0)
- moved P4 58.1 mm to (70.0, 58.0)
- moved P7 56.7 mm to (27.0, 21.0)
- moved P3 36.1 mm to (18.0, 54.0)
- moved P6 34.2 mm to (113.0, 21.0)
- moved SW12 2.00 mm to (18.0, 21.0)
- moved SW13 2.00 mm to (36.0, 21.0)
- moved SW14 2.00 mm to (104.0, 21.0)
- moved SW15 2.00 mm to (122.0, 21.0)
- moved L4 1.65 mm to (94.4, 40.0)
- moved U2 1.53 mm to (90.3, 38.9)
- moved C14 1.52 mm to (90.2, 36.4)
- moved C15 1.52 mm to (90.3, 41.1)
- moved Q1 1.52 mm to (94.2, 35.8)
- moved BATT1 1.50 mm to (93.5, 33.0)
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Connections:
- net /Input/A renamed /A
- net /Input/B renamed /B
- net /Input/DOWN renamed /DOWN
- net /Input/HOME renamed /HOME
- net /Input/LEFT renamed /LEFT
- net /Input/LS renamed /JS_LS
- net /Input/LX renamed /JS_LX
- net /Input/LY renamed /JS_LY
- net /Input/RIGHT renamed /RIGHT
- net /Input/RS renamed /JS_RS
- net /Input/RX renamed /JS_RX
- net /Input/RY renamed /JS_RY
- net /Input/SELECT renamed /SELECT
- net /Input/START renamed /START
- net /Input/UP renamed /UP
- net /Input/X renamed /X
- net /Input/Y renamed /Y
- net Net-(P11-Pad1) renamed /GND_R
- net Net-(P8-Pad1) renamed /GND_L
- SH_L1 pad 1: +3V3 -> /L1
- SH_L1 pad 2: /Input/L1 -> /L2
- SH_L1 pad 3: /Input/L2 -> GND
- SH_R1 pad 1: /Input/R2 -> GND
- SH_R1 pad 2: /Input/R1 -> /R2
- SH_R1 pad 3: +3V3 -> /R1
- SW1 pad 1: +3V3 -> GND
- SW10 pad 1: +3V3 -> GND
- SW11 pad 1: +3V3 -> GND
- SW2 pad 1: +3V3 -> GND
- SW3 pad 1: +3V3 -> GND
- SW4 pad 1: +3V3 -> GND
- SW5 pad 1: +3V3 -> GND
- SW6 pad 1: +3V3 -> GND
- SW7 pad 1: +3V3 -> GND
- SW8 pad 1: +3V3 -> GND
- SW9 pad 1: +3V3 -> GND
- U1 pad 33: /Input/L2 -> /L2
- U1 pad 34: /Input/L1 -> /L1
- U1 pad 4: /Input/R1 -> /R1
- U1 pad 5: /Input/R2 -> /R2
Routing:
- net +3V3: track 298.4 -> 137.7 mm
- net /GND_L: track 36.5 -> 0.00 mm
- net /GND_R: track 36.4 -> 0.00 mm
- net /Input/R2: track 35.2 -> 0.00 mm
- net /Input/L2: track 34.9 -> 0.00 mm
- net /Input/R1: track 34.6 -> 0.00 mm
- net /Input/L1: track 34.2 -> 0.00 mm
- net /L2: track 0.00 -> 30.0 mm
- net /R2: track 0.00 -> 29.8 mm
- net /L1: track 0.00 -> 28.2 mm
- net /R1: track 0.00 -> 28.0 mm
- net /HOME: track 22.8 -> 3.75 mm
- net /LEFT: track 55.3 -> 41.5 mm
- net /SELECT: track 28.2 -> 14.8 mm
- net /DOWN: track 51.0 -> 38.3 mm
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- added copper zone on F.Cu, net /GND_L
- added copper zone on F.Cu, net /GND_R
- removed copper zone on F.Cu, net (none)
Other:
- board size 114 x 50 mm -> 114 x 48 mm
