File: Controller/Input.sch (KiCad schematic (older format))
At the start: 36 parts, among them P11 CONN_SHOULDER, P8 CONN_SHOULDER, SW1 BUTTON, SW10 BUTTON, SW11 BUTTON, SW12 BUTTON, SW13 BUTTON, SW14 BUTTON, SW15 BUTTON, SW2 BUTTON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

Commit message: Improved traces in power supply circuit. Added clearance on inside of drill holes. Removed sharp inside corners and replaced with cirular cutouts. Removed removed pull-down resistors because I am using internal pull-ups and negative logic with buttons.
Parts:
- removed R10, R11, R12, R13, R14, R15, R16, R17, R18, R19, R20: 10k, Resistors_SMD:R_0805, symbol 10k
Connections:
- net +3V3: no longer SW1.1, SW10.1, SW11.1, SW2.1, SW3.1, SW4.1, SW5.1, SW6.1, SW7.1, SW8.1, SW9.1
- net GND: now also SW1.1, SW10.1, SW11.1, SW2.1, SW3.1, SW4.1, SW5.1, SW6.1, SW7.1, SW8.1, SW9.1
Other:
- note added: "I will use the NRF51822's\ninternal pull-up resistors"
